File: pcb/mainboardx2/mainboardx2.kicad_pcb (KiCad board)
At the start: 2 copper layers, 150 x 150 mm, 31 parts, among them J1 Compass, J10 Right, J11 Back, J12 Conn_01x03_Socket, J13 Conn_01x03_Socket, J14 Conn_01x03_Socket, J15 Conn_01x03_Socket, J16 Conn_01x03_Socket, J17 Conn_01x03_Socket, J18 Conn_01x03_Socket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

Commit message: pins remapping
Parts:
- added U1: AMS1117-3.3, Package_TO_SOT_SMD:SOT-223-3_TabPin2, B.Cu at (117.6, 67.7)
Connections:
- J3 pad 19: +3.3V -> unconnected-(J3-Pin_19-Pad19)
- J4 pad 1: GND -> +3.3V
- J4 pad 2: +3.3V -> GND
Routing:
- net GND: track 745.9 -> 766.6 mm
- net +3.3V: track 483.3 -> 492.4 mm
- net +5V: track 183.8 -> 189.9 mm
