File: pcb/cam/cam.kicad_sch (KiCad schematic)
At the start: 14 parts

Commit message: init
Parts:
- renumbered CAM_1 to CAM1_
Changed lines of the file:
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@@
 	(generator_version "9.0")
 	(paper "A4")
+	(rectangle
+		(start 74.93 48.26)
+		(end 105.41 69.85)
+		(stroke
+			(width 0)
+			(type default)
+		)
+		(fill
+			(type none)
+		)
+	)
 	(junction
 		(at 110.49 92.71)
@@
 		(on_board yes)
 		(dnp no)
-		(property "Reference" "CAM_1"
+		(property "Reference" "CAM1_"
 			(at 104.14 58.42 0)
 			(effects
@@
 			(project ""
 				(path "/6ec8a7a2-ab39-4f77-8961-49439b5813eb"
-					(reference "CAM_1")
+					(reference "CAM1_")
 					(unit 1)
 				)
