File: pcb/mainboard/mainboard.kicad_pcb (KiCad board)
At the start: 2 copper layers, 150 x 150 mm, 34 parts, among them J1 Compass, J10 Right, J11 Back, J12 Conn_01x03_Socket, J13 Conn_01x03_Socket, J14 Conn_01x03_Socket, J15 Conn_01x03_Socket, J16 Conn_01x03_Socket, J17 Conn_01x03_Socket, J18 Conn_01x03_Socket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

Commit message: fixup
Parts:
- added SW2: Set, Diode_THT:D_5W_P5.08mm_Vertical_AnodeUp, F.Cu at (149.9, 91.4)
- REF**: value PinSocket_1x08_P2.54mm_Vertical -> PinSocket_1x07_P2.54mm_Vertical; footprint Connector_PinSocket_2.54mm:PinSocket_1x08_P2.54mm_Vertical -> Connector_PinSocket_2.54mm:PinSocket_1x07_P2.54mm_Vertical
Connections:
- J3 pad 12: unconnected-(J3-Pin_12-Pad12) -> Net-(J3-Pin_12)
Routing:
- net Net-(J3-Pin_12): track 0.00 -> 32.6 mm
- net unconnected-(J3-Pin_12-Pad12): track 5.08 -> 0.00 mm
- net Net-(J2-Pin_14): track 91.9 -> 95.2 mm
- net Net-(J2-Pin_11): track 88.7 -> 92.0 mm

Commit message: linesensor
Parts:
- SW2: value Set -> Mode
Connections:
- J9 pad 3: Net-(J2-Pin_10) -> Net-(J3-Pin_12)
- SW2 pad 1: Net-(J3-Pin_12) -> Net-(J2-Pin_10)
Routing:
- net Net-(J2-Pin_10): track 40.8 -> 0.00 mm
- net Net-(J3-Pin_12): track 32.6 -> 0.00 mm
Changed lines of the file:
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@@
 			(layers "*.Cu" "*.Mask")
 			(remove_unused_layers no)
-			(net 19 "Net-(J2-Pin_10)")
+			(net 51 "Net-(J3-Pin_12)")
 			(pinfunction "Pin_3")
 			(pintype "passive")
@@
 			)
 		)
-		(property "Value" "Set"
+		(property "Value" "Mode"
 			(at 2.54 3.174899 90)
 			(layer "F.Fab")
@@
 			(layers "*.Cu" "*.Mask")
 			(remove_unused_layers no)
-			(net 51 "Net-(J3-Pin_12)")
+			(net 19 "Net-(J2-Pin_10)")
 			(pinfunction "1")
 			(pintype "passive")
@@
 	)
 	(segment
-		(start 104.14 73.66)
-		(end 123.698 93.218)
-		(width 1)
-		(layer "B.Cu")
-		(net 19)
-	)
-	(segment
-		(start 123.698 99.712213)
-		(end 125.585787 101.6)
-		(width 1)
-		(layer "B.Cu")
-		(net 19)
-	)
-	(segment
-		(start 123.698 93.218)
-		(end 123.698 99.712213)
-		(width 1)
-		(layer "B.Cu")
-		(net 19)
-	)
-	(segment
-		(start 101.6 73.66)
-		(end 104.14 73.66)
-		(width 1)
-		(layer "B.Cu")
-		(net 19)
-	)
-	(segment
-		(start 125.585787 101.6)
-		(end 127 101.6)
-		(width 1)
-		(layer "B.Cu")
-		(net 19)
-	)
-	(segment
 		(start 111.76 96.52)
 		(end 111.76 99.06)
@@
 		(net 50)
 	)
-	(segment
-		(start 147.32 88.9)
-		(end 149.86 91.44)
-		(width 1)
-		(layer "B.Cu")
-		(net 51)
-	)
-	(segment
-		(start 127 78.74)
-		(end 144.78 78.74)
-		(width 1)
-		(layer "B.Cu")
-		(net 51)
-	)
-	(segment
-		(start 144.78 78.74)
-		(end 147.32 81.28)
-		(width 1)
-		(layer "B.Cu")
-		(net 51)
-	)
-	(segment
-		(start 147.32 81.28)
-		(end 147.32 88.9)
-		(width 1)
-		(layer "B.Cu")
-		(net 51)
-	)
 	(zone
