File: pcb/mainboard/mainboard.kicad_sch (KiCad schematic)
At the start: 27 parts, among them J1 Compass, J10 Right, J11 Back, J12 Conn_01x03_Socket, J13 Conn_01x03_Socket, J14 Conn_01x03_Socket, J15 Conn_01x03_Socket, J16 Conn_01x03_Socket, J17 Conn_01x03_Socket, J18 Conn_01x03_Socket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

Commit message: fixup
Parts:
- added SW2: Set, Diode_THT:D_5W_P5.08mm_Vertical_AnodeUp, symbol Switch:SW_Push
Connections:
- net GND: now also SW2.2
- net at J3.12 (Pin_12): now also SW2.1
Changed lines of the file:
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@@
+	(wire
+		(pts
+			(xy 148.59 76.2) (xy 161.29 76.2)
+		)
+		(stroke
+			(width 0)
+			(type default)
+		)
+	)
 	(wire
 		(pts
@@
 	(wire
 		(pts
+			(xy 161.29 95.25) (xy 186.69 95.25)
+		)
+		(stroke
+			(width 0)
+			(type default)
+		)
+	)
+	(wire
+		(pts
 			(xy 160.02 96.52) (xy 180.34 96.52)
 		)
@@
 	(wire
 		(pts
+			(xy 196.85 96.52) (xy 196.85 97.79)
+		)
+		(stroke
+			(width 0)
+			(type default)
+		)
+	)
+	(wire
+		(pts
 			(xy 90.17 80.01) (xy 90.17 81.28)
 		)
@@
 	(wire
 		(pts
+			(xy 186.69 95.25) (xy 186.69 96.52)
+		)
+		(stroke
+			(width 0)
+			(type default)
+		)
+	)
+	(wire
+		(pts
 			(xy 96.52 105.41) (xy 96.52 111.76)
 		)
@@
 		(pts
 			(xy 128.27 83.82) (xy 129.54 83.82)
+		)
+		(stroke
+			(width 0)
+			(type default)
+		)
+	)
+	(wire
+		(pts
+			(xy 161.29 76.2) (xy 161.29 95.25)
 		)
 		(stroke
@@
 					(unit 1)
 				)
+			)
+		)
+	)
+	(symbol
+		(lib_id "power:GND")
+		(at 196.85 97.79 0)
+		(unit 1)
+		(exclude_from_sim no)
+		(in_bom yes)
+		(on_board yes)
+		(dnp no)
+		(fields_autoplaced yes)
+		(property "Reference" "#PWR017"
+			(at 196.85 104.14 0)
+			(effects
+				(font
+					(size 1.27 1.27)
+				)
+				(hide yes)
+			)
+		)
+		(property "Value" "GND"
+			(at 196.85 102.87 0)
+			(effects
+				(font
+					(size 1.27 1.27)
+				)
+			)
+		)
+		(property "Footprint" ""
+			(at 196.85 97.79 0)
+			(effects
+				(font
+					(size 1.27 1.27)
+				)
+				(hide yes)
+			)
+		)
+		(property "Datasheet" ""
+			(at 196.85 97.79 0)
+			(effects
+				(font
+					(size 1.27 1.27)
+				)
+				(hide yes)
+			)
+		)
+		(property "Description" "Power symbol creates a global label with name \"GND\" , ground"
+			(at 196.85 97.79 0)
+			(effects
+				(font
+					(size 1.27 1.27)
+				)
+				(hide yes)
+			)
+		)
+		(pin "1"
+		)
+		(instances
+			(project "mainboard"
+				(path "/5ae74e10-1887-43ae-95c4-acccf3a5a562"
+					(reference "#PWR017")
+					(unit 1)
+				)
+			)
+		)
+	)
+	(symbol
+		(lib_id "Switch:SW_Push")
+		(at 191.77 96.52 0)
+		(unit 1)
+		(exclude_from_sim no)
+		(in_bom yes)
+		(on_board yes)
+		(dnp no)
+		(fields_autoplaced yes)
+		(property "Reference" "SW2"
+			(at 191.77 88.9 0)
+			(effects
+				(font
+					(size 1.27 1.27)
+				)
+			)
+		)
+		(property "Value" "Set"
+			(at 191.77 91.44 0)
+			(effects
+				(font
+					(size 1.27 1.27)
+				)
+			)
+		)
+		(property "Footprint" "Diode_THT:D_5W_P5.08mm_Vertical_AnodeUp"
+			(at 191.77 91.44 0)
+			(effects
+				(font
+					(size 1.27 1.27)
+				)
+				(hide yes)
+			)
+		)
+		(property "Datasheet" "~"
+			(at 191.77 91.44 0)
+			(effects
+				(font
+					(size 1.27 1.27)
+				)
+				(hide yes)
+			)
+		)
+		(property "Description" "Push button switch, generic, two pins"
+			(at 191.77 96.52 0)
+			(effects
+				(font
+					(size 1.27 1.27)
+				)
+				(hide yes)
+			)
+		)
+		(pin "2"
+		)
+		(pin "1"
+		)
+		(instances
+			(project "mainboard"
+				(path "/5ae74e10-1887-43ae-95c4-acccf3a5a562"
+					(reference "SW2")
+					(unit 1)
+				)

Commit message: IR ring
Parts:
- SW2: value Set -> Mode
Connections:
- net at J9.3 (Pin_3): now also J3.12 (Pin_12); no longer J2.10 (Pin_10)
- net at SW2.1: now also J2.10 (Pin_10); no longer J3.12 (Pin_12)
Other:
- moved on the sheet: J10, J11, J9, SW1, SW2

Commit message: mainboard scheme update
Connections:
- net at J1.6 (Pin_6): now also J3.6 (Pin_6); no longer J3.3 (Pin_3)
- net at J1.7 (Pin_7): now also J3.5 (Pin_5); no longer J3.4 (Pin_4)
- net at J3.7 (Pin_7): now also J5.1 (Pin_1)
- net key: now reaches J3.8 (Pin_8)
- net at J2.3 (Pin_3): no longer J5.1 (Pin_1)
- no-connect marks 0 -> 3
